File: hardware/ki_cad/daughter_boards/relay/relay_daughter/relay_daughter.kicad_sch (KiCad schematic)
At the start: 6 parts, among them J1 ToMainPCB, K1 SANYOU_SRD_Form_A, K2 SANYOU_SRD_Form_A

Commit message: relay daughter PCB frozen, Unisync story frozen
Parts:
- removed K1, K2: SANYOU_SRD_Form_A, Relay_THT:Relay_SPST_SANYOU_SRD_Series_Form_A, symbol Relay:SANYOU_SRD_Form_A
- added K3, K4: SANYOU_SRD_Form_C, Relay_THT:Relay_SPDT_SANYOU_SRD_Series_Form_C, symbol Relay:SANYOU_SRD_Form_C
- C_SNUB1, C_SNUB2: footprint Capacitor_THT:C_Disc_D7.0mm_W2.5mm_P5.00mm -> Capacitor_THT:C_Rect_L18.0mm_W5.0mm_P15.00mm_FKS3_FKP3
Connections:
- net +5V: now also K3.5, K4.5
- net LOAD_OUT1: now also K4.1
- net LOAD_OUT2: now also TB1.3 (Pin_3), K3.1; no longer TB1.2 (Pin_2)
- net MAINS_LIVE_IN1: now also TB1.2 (Pin_2), K3.3, K4.3; no longer TB1.3 (Pin_3)
- net RELAY_OUT1: now also K4.2
- net RELAY_OUT2: now also K3.2
- no-connect marks 0 -> 2
